Commit message: urdf changed

File: frobo_description/urdf/frobo.urdf.xacro (robot description, xacro)
@@ -17,5 +17,5 @@
   <!-- uarm -->
   <uarm color="Black" parent="base_link">
-    <origin xyz="0.015 0 0.137" rpy="0 0 0"/>
+    <origin xyz="0.015 0 0.137" rpy="0 0 ${M_PI}"/>
   </uarm>
   <!-- Camera -->

File: frobo_description/urdf/uarm.urdf.xacro (robot description, xacro)
@@ -1,12 +1,12 @@
 <?xml version="1.0"?>
 <robot xmlns:xacro="http://www.ros.org/wiki/xacro">
- <!-- define a sonar -->
+ <!-- uArm description -->
   <xacro:macro name="uarm" params="parent  color *origin">
     <joint name="uarm_joint" type="fixed">
       <xacro:insert_block name="origin" />
       <parent link="${parent}"/>
-      <child link="uarm_link"/>
+      <child link="uarm_base_link"/>
     </joint>
-    <link name="uarm_link">
+    <link name="uarm_base_link">
       <visual>
         <origin xyz="0 0 0" rpy="0 0 0" />
@@ -17,4 +17,102 @@
       </visual>
     </link>
+    <joint name="uarm_base_body_joint" type="continuous">
+      <origin xyz="0 0 0.01" rpy="0 0 0"/>
+      <parent link="uarm_base_link"/>
+      <child link="uarm_body_link"/>
+    </joint>
+    <link name="uarm_body_link">
+      <visual>
+        <origin xyz="0 0 -0.01" rpy="0 0 0" />
+        <geometry>
+            <mesh filename="package://frobo_description/meshes/uarm_body.stl" scale="0.001 0.001 0.001"/>
+        </geometry>
+        <material name="${color}" />
+      </visual>
+    </link>
+    <joint name="uarm_body_upper_arm_joint" type="continuous">
+      <origin xyz="-0.02 0 0.07" rpy="0 0 0"/>
+      <parent link="uarm_body_link"/>
+      <child link="uarm_upper_arm_link"/>
+    </joint>
+    <link name="uarm_upper_arm_link">
+      <visual>
+        <origin xyz="0.02 0 -${0.07+0.01}" rpy="0 0 0" />
+        <geometry>
+            <mesh filename="package://frobo_description/meshes/uarm_upper_arm.stl" scale="0.001 0.001 0.001"/>
+        </geometry>
+        <material name="${color}" />
+      </visual>
+    </link>
+    <joint name="uarm_upper_arm_forearm_joint" type="continuous">
+      <origin xyz="0.048 0 0.138" rpy="0 0 0"/>
+      <parent link="uarm_upper_arm_link"/>
+      <child link="uarm_forearm_link"/>
+    </joint>
+   <link name="uarm_forearm_link">
+      <visual>
+        <origin xyz="-${-0.02+0.048} 0 -${0.07+0.01+0.138}" rpy="0 0 0" />
+        <geometry>
+            <mesh filename="package://frobo_description/meshes/uarm_forearm.stl" scale="0.001 0.001 0.001"/>
+        </geometry>
+        <material name="${color}" />
+      </visual>
+    </link>
+    <joint name="uarm_forearm_palm_holder_joint" type="continuous">
+      <origin xyz="-0.145 0 -0.068" rpy="0 0 0"/>
+      <parent link="uarm_forearm_link"/>
+      <child link="uarm_palm_holder_link"/>
+    </joint>
+    <link name="uarm_palm_holder_link">
+      <visual>
+        <origin xyz="${-(-0.02+0.048-0.145)} 0 ${-(0.07+0.01+0.138-0.068)}" rpy="0 0 0" />
+        <geometry>
+            <mesh filename="package://frobo_description/meshes/uarm_palm_holder.stl" scale="0.001 0.001 0.001"/>
+        </geometry>
+        <material name="${color}" />
+      </visual>
+    </link>
+    <joint name="palm_holder_palm_joint" type="continuous">
+      <origin xyz="-0.036 -0.0029 -0.011" rpy="0 0 0"/>
+      <parent link="uarm_palm_holder_link"/>
+      <child link="uarm_palm_link"/>
+    </joint>
+    <link name="uarm_palm_link">
+      <visual>
+        <origin xyz="0.009 0 0" rpy="${-M_PI/2} 0 ${M_PI/2}" />
+        <geometry>
+            <mesh filename="package://frobo_description/meshes/uarm_palm.stl" scale="0.001 0.001 0.001"/>
+        </geometry>
+        <material name="${color}" />
+      </visual>
+    </link>
+    <joint name="palm_left_finger_joint" type="continuous">
+      <origin xyz="0 -0.008 -0.035" rpy="0 0 0"/>
+      <parent link="uarm_palm_link"/>
+      <child link="uarm_left_finger_link"/>
+    </joint>
+    <link name="uarm_left_finger_link">
+      <visual>
+        <origin xyz="0.009 0.008 0.035" rpy="${-M_PI/2} 0 ${M_PI/2}" />
+        <geometry>
+            <mesh filename="package://frobo_description/meshes/uarm_left_finger.stl" scale="0.001 0.001 0.001"/>
+        </geometry>
+        <material name="${color}" />
+      </visual>
+    </link>
+    <joint name="palm_right_finger_joint" type="continuous">
+      <origin xyz="0 0.008 -0.035" rpy="0 0 0"/>
+      <parent link="uarm_palm_link"/>
+      <child link="uarm_right_finger_link"/>
+    </joint>
+    <link name="uarm_right_finger_link">
+      <visual>
+        <origin xyz="0.009 -0.008 0.035" rpy="${-M_PI/2} 0 ${M_PI/2}" />
+        <geometry>
+            <mesh filename="package://frobo_description/meshes/uarm_right_finger.stl" scale="0.001 0.001 0.001"/>
+        </geometry>
+        <material name="${color}" />
+      </visual>
+    </link>
   </xacro:macro>
 </robot>
